Commit message: 1.0.7 Add the TM5S and TM7S, mesh files and Xacro simulation models.

File: tm_description/xacro/macro.tm5s-nominal.urdf.xacro (robot description, xacro)
@@ -2,19 +2,19 @@
 <robot xmlns:xacro="http://www.ros.org/wiki/xacro">
   <xacro:include filename="$(find tm_description)/xacro/macro.inertial.xacro" />
-  <xacro:macro name="tm12s" params="ns prefix color:=none format:=obj
+  <xacro:macro name="tm5s" params="ns prefix color:=none format:=obj
     shoulder_1_joint_lower_limit:=${radians(-360)}    shoulder_1_joint_upper_limit:=${radians(360)}
     shoulder_2_joint_lower_limit:=${radians(-360)}    shoulder_2_joint_upper_limit:=${radians(360)}
-    elbow_joint_lower_limit:=${radians(-162)}    elbow_joint_upper_limit:=${radians(162)}
+    elbow_joint_lower_limit:=${radians(-158)}    elbow_joint_upper_limit:=${radians(158)}
     wrist_1_joint_lower_limit:=${radians(-360)}    wrist_1_joint_upper_limit:=${radians(360)}
     wrist_2_joint_lower_limit:=${radians(-360)}    wrist_2_joint_upper_limit:=${radians(360)}
     wrist_3_joint_lower_limit:=${radians(-360)}    wrist_3_joint_upper_limit:=${radians(360)}
-    shoulder_1_joint_velocity_limit:=${radians(160)}
-    shoulder_2_joint_velocity_limit:=${radians(160)}
+    shoulder_1_joint_velocity_limit:=${radians(240)}
+    shoulder_2_joint_velocity_limit:=${radians(240)}
     elbow_joint_velocity_limit:=${radians(240)}
     wrist_1_joint_velocity_limit:=${radians(260)}
     wrist_2_joint_velocity_limit:=${radians(260)}
     wrist_3_joint_velocity_limit:=${radians(520)}
-    shoulder_1_joint_effort_limit:=${350}
-    shoulder_2_joint_effort_limit:=${350}
+    shoulder_1_joint_effort_limit:=${170}
+    shoulder_2_joint_effort_limit:=${170}
     elbow_joint_effort_limit:=${170}
     wrist_1_joint_effort_limit:=${45}
@@ -39,26 +39,26 @@
     <!-- Inertia parameters -->
     <xacro:property name="mass_0" value="1.0" />
-    <xacro:property name="mass_1" value="8.200" />
-    <xacro:property name="mass_2" value="15.017" />
-    <xacro:property name="mass_3" value="3.329" />
+    <xacro:property name="mass_1" value="4.320" />
+    <xacro:property name="mass_2" value="9.796" />
+    <xacro:property name="mass_3" value="2.778" />
     <xacro:property name="mass_4" value="1.770" />
-    <xacro:property name="mass_5" value="1.880" />
+    <xacro:property name="mass_5" value="1.770" />
     <xacro:property name="mass_6" value="0.720" />
     <xacro:property name="unit_factor" value="0.000001"/>
-    <xacro:property name="ixx_1" value="${25963.078*unit_factor}" />
-    <xacro:property name="ixx_2" value="${56178.979*unit_factor}" />
-    <xacro:property name="ixx_3" value="${4694.5431*unit_factor}" />
+    <xacro:property name="ixx_1" value="${8439.2993*unit_factor}" />
+    <xacro:property name="ixx_2" value="${29227.499*unit_factor}" />
+    <xacro:property name="ixx_3" value="${4173.2753*unit_factor}" />
     <xacro:property name="ixx_4" value="${2046.0318*unit_factor}" />
     <xacro:property name="ixx_5" value="${2046.0318*unit_factor}" />
     <xacro:property name="ixx_6" value="${703.44734*unit_factor}" />
-    <xacro:property name="iyy_1" value="${37671.229*unit_factor}" />
-    <xacro:property name="iyy_2" value="${1212610.4*unit_factor}" />
-    <xacro:property name="iyy_3" value="${134098.54*unit_factor}" />
+    <xacro:property name="iyy_1" value="${13793.964*unit_factor}" />
+    <xacro:property name="iyy_2" value="${406910.57*unit_factor}" />
+    <xacro:property name="iyy_3" value="${61909.685*unit_factor}" />
     <xacro:property name="iyy_4" value="${3171.8293*unit_factor}" />
     <xacro:property name="iyy_5" value="${3171.8293*unit_factor}" />
     <xacro:property name="iyy_6" value="${1711.0225*unit_factor}" />
-    <xacro:property name="izz_1" value="${38856.370*unit_factor}" />
-    <xacro:property name="izz_2" value="${1231270.0*unit_factor}" />
-    <xacro:property name="izz_3" value="${135525.91*unit_factor}" />
+    <xacro:property name="izz_1" value="${14241.226*unit_factor}" />
+    <xacro:property name="izz_2" value="${418507.58*unit_factor}" />
+    <xacro:property name="izz_3" value="${63318.609*unit_factor}" />
     <xacro:property name="izz_4" value="${3478.9518*unit_factor}" />
     <xacro:property name="izz_5" value="${3478.9518*unit_factor}" />
@@ -68,11 +68,11 @@
     <visual>
       <geometry>
-        <mesh filename="package://tm_description/meshes/tm12s/visual/tm12s-tbb_a.${format}" />
-      </geometry>
-      <material name="${color}" />
-    </visual>
-    <collision>
-      <geometry>
-        <mesh filename="package://tm_description/meshes/tm12s/collision/tm12s-tbb_a_c.stl" />
+        <mesh filename="package://tm_description/meshes/tm5s/visual/tm5s-base.${format}" />
+      </geometry>
+      <material name="${color}" />
+    </visual>
+    <collision>
+      <geometry>
+        <mesh filename="package://tm_description/meshes/tm5s/collision/tm5s-base_c.stl" />
       </geometry>
     </collision>
@@ -85,5 +85,5 @@
     <parent link="${prefix}link_0" />
     <child link="${prefix}link_1" />
-    <origin rpy="0.000000 -0.000000 0.000000" xyz="0.000000 0.000000 0.165200" />
+    <origin rpy="0.000000 -0.000000 0.000000" xyz="0.000000 0.000000 0.148400" />
     <axis xyz="0 0 1" />
 <!--limit-->
@@ -97,11 +97,11 @@
     <visual>
       <geometry>
-        <mesh filename="package://tm_description/meshes/tm12s/visual/tm12s-j1-a.${format}" />
-      </geometry>
-      <material name="${color}" />
-    </visual>
-    <collision>
-      <geometry>
-        <mesh filename="package://tm_description/meshes/tm12s/collision/tm12s-j1-a_c.stl" />
+        <mesh filename="package://tm_description/meshes/tm5s/visual/tm5s-j1.${format}" />
+      </geometry>
+      <material name="${color}" />
+    </visual>
+    <collision>
+      <geometry>
+        <mesh filename="package://tm_description/meshes/tm5s/collision/tm5s-j1_c.stl" />
       </geometry>
     </collision>
@@ -127,11 +127,11 @@
     <visual>
       <geometry>
-        <mesh filename="package://tm_description/meshes/tm12s/visual/tm12s-a1.${format}" />
-      </geometry>
-      <material name="${color}" />
-    </visual>
-    <collision>
-      <geometry>
-        <mesh filename="package://tm_description/meshes/tm12s/collision/tm12s-a1_c.stl" />
+        <mesh filename="package://tm_description/meshes/tm5s/visual/tm5s-a1.${format}" />
+      </geometry>
+      <material name="${color}" />
+    </visual>
+    <collision>
+      <geometry>
+        <mesh filename="package://tm_description/meshes/tm5s/collision/tm5s-a1_c.stl" />
       </geometry>
     </collision>
@@ -145,5 +145,5 @@
     <parent link="${prefix}link_2" />
     <child link="${prefix}link_3" />
-    <origin rpy="0.000000 -0.000000 0.000000" xyz="0.636100 0.000000 0.000000" />
+    <origin rpy="0.000000 -0.000000 0.000000" xyz="0.429000 0.000000 0.000000" />
     <axis xyz="0 0 1" />
 <!--limit-->
@@ -157,11 +157,11 @@
     <visual>
       <geometry>
-        <mesh filename="package://tm_description/meshes/tm12s/visual/tm12s-a2.${format}" />
-      </geometry>
-      <material name="${color}" />
-    </visual>
-    <collision>
-      <geometry>
-        <mesh filename="package://tm_description/meshes/tm12s/collision/tm12s-a2_c.stl" />
+        <mesh filename="package://tm_description/meshes/tm5s/visual/tm5s-a2.${format}" />
+      </geometry>
+      <material name="${color}" />
+    </visual>
+    <collision>
+      <geometry>
+        <mesh filename="package://tm_description/meshes/tm5s/collision/tm5s-a2_c.stl" />
       </geometry>
     </collision>
@@ -175,5 +175,5 @@
     <parent link="${prefix}link_3" />
     <child link="${prefix}link_4" />
-    <origin rpy="0.000000 -0.000000 1.570796" xyz="0.532400 0.000000 -0.181800" />
+    <origin rpy="0.000000 -0.000000 1.570796" xyz="0.386000 0.000000 -0.147800" />
     <axis xyz="0 0 1" />
 <!--limit-->
@@ -187,11 +187,11 @@
     <visual>
       <geometry>
-        <mesh filename="package://tm_description/meshes/tm12s/visual/tm12s-j5.${format}" />
-      </geometry>
-      <material name="${color}" />
-    </visual>
-    <collision>
-      <geometry>
-        <mesh filename="package://tm_description/meshes/tm12s/collision/tm12s-j5_c.stl" />
+        <mesh filename="package://tm_description/meshes/tm5s/visual/tm5s-j5.${format}" />
+      </geometry>
+      <material name="${color}" />
+    </visual>
+    <collision>
+      <geometry>
+        <mesh filename="package://tm_description/meshes/tm5s/collision/tm5s-j5_c.stl" />
       </geometry>
     </collision>
@@ -217,11 +217,11 @@
     <visual>
       <geometry>
-        <mesh filename="package://tm_description/meshes/tm12s/visual/tm12s-j6.${format}" />
-      </geometry>
-      <material name="${color}" />
-    </visual>
-    <collision>
-      <geometry>
-        <mesh filename="package://tm_description/meshes/tm12s/collision/tm12s-j6_c.stl" />
+        <mesh filename="package://tm_description/meshes/tm5s/visual/tm5s-j6.${format}" />
+      </geometry>
+      <material name="${color}" />
+    </visual>
+    <collision>
+      <geometry>
+        <mesh filename="package://tm_description/meshes/tm5s/collision/tm5s-j6_c.stl" />
       </geometry>
     </collision>
@@ -247,11 +247,11 @@
     <visual>
       <geometry>
-        <mesh filename="package://tm_description/meshes/tm12s/visual/tm12s-io.${format}" />
-      </geometry>
-      <material name="${color}" />
-    </visual>
-    <collision>
-      <geometry>
-        <mesh filename="package://tm_description/meshes/tm12s/collision/tm12s-io_c.stl" />
+        <mesh filename="package://tm_description/meshes/tm5s/visual/tm5s-io.${format}" />
+      </geometry>
+      <material name="${color}" />
+    </visual>
+    <collision>
+      <geometry>
+        <mesh filename="package://tm_description/meshes/tm5s/collision/tm5s-io_c.stl" />
       </geometry>
     </collision>

File: tm_description/xacro/macro.tm7s-nominal.urdf.xacro (robot description, xacro)
@@ -2,19 +2,19 @@
 <robot xmlns:xacro="http://www.ros.org/wiki/xacro">
   <xacro:include filename="$(find tm_description)/xacro/macro.inertial.xacro" />
-  <xacro:macro name="tm12s" params="ns prefix color:=none format:=obj
+  <xacro:macro name="tm7s" params="ns prefix color:=none format:=obj
     shoulder_1_joint_lower_limit:=${radians(-360)}    shoulder_1_joint_upper_limit:=${radians(360)}
     shoulder_2_joint_lower_limit:=${radians(-360)}    shoulder_2_joint_upper_limit:=${radians(360)}
-    elbow_joint_lower_limit:=${radians(-162)}    elbow_joint_upper_limit:=${radians(162)}
+    elbow_joint_lower_limit:=${radians(-152)}    elbow_joint_upper_limit:=${radians(152)}
     wrist_1_joint_lower_limit:=${radians(-360)}    wrist_1_joint_upper_limit:=${radians(360)}
     wrist_2_joint_lower_limit:=${radians(-360)}    wrist_2_joint_upper_limit:=${radians(360)}
     wrist_3_joint_lower_limit:=${radians(-360)}    wrist_3_joint_upper_limit:=${radians(360)}
-    shoulder_1_joint_velocity_limit:=${radians(160)}
-    shoulder_2_joint_velocity_limit:=${radians(160)}
+    shoulder_1_joint_velocity_limit:=${radians(240)}
+    shoulder_2_joint_velocity_limit:=${radians(240)}
     elbow_joint_velocity_limit:=${radians(240)}
     wrist_1_joint_velocity_limit:=${radians(260)}
     wrist_2_joint_velocity_limit:=${radians(260)}
     wrist_3_joint_velocity_limit:=${radians(520)}
-    shoulder_1_joint_effort_limit:=${350}
-    shoulder_2_joint_effort_limit:=${350}
+    shoulder_1_joint_effort_limit:=${170}
+    shoulder_2_joint_effort_limit:=${170}
     elbow_joint_effort_limit:=${170}
     wrist_1_joint_effort_limit:=${45}
@@ -39,26 +39,26 @@
     <!-- Inertia parameters -->
     <xacro:property name="mass_0" value="1.0" />
-    <xacro:property name="mass_1" value="8.200" />
-    <xacro:property name="mass_2" value="15.017" />
-    <xacro:property name="mass_3" value="3.329" />
+    <xacro:property name="mass_1" value="4.320" />
+    <xacro:property name="mass_2" value="9.456" />
+    <xacro:property name="mass_3" value="2.618" />
     <xacro:property name="mass_4" value="1.770" />
-    <xacro:property name="mass_5" value="1.880" />
+    <xacro:property name="mass_5" value="1.770" />
     <xacro:property name="mass_6" value="0.720" />
     <xacro:property name="unit_factor" value="0.000001"/>
-    <xacro:property name="ixx_1" value="${25963.078*unit_factor}" />
-    <xacro:property name="ixx_2" value="${56178.979*unit_factor}" />
-    <xacro:property name="ixx_3" value="${4694.5431*unit_factor}" />
+    <xacro:property name="ixx_1" value="${8439.2993*unit_factor}" />
+    <xacro:property name="ixx_2" value="${28756.423*unit_factor}" />
+    <xacro:property name="ixx_3" value="${4027.8840*unit_factor}" />
     <xacro:property name="ixx_4" value="${2046.0318*unit_factor}" />
     <xacro:property name="ixx_5" value="${2046.0318*unit_factor}" />
     <xacro:property name="ixx_6" value="${703.44734*unit_factor}" />
-    <xacro:property name="iyy_1" value="${37671.229*unit_factor}" />
-    <xacro:property name="iyy_2" value="${1212610.4*unit_factor}" />
-    <xacro:property name="iyy_3" value="${134098.54*unit_factor}" />
+    <xacro:property name="iyy_1" value="${13793.964*unit_factor}" />
+    <xacro:property name="iyy_2" value="${240700.11*unit_factor}" />
+    <xacro:property name="iyy_3" value="${35507.262*unit_factor}" />
     <xacro:property name="iyy_4" value="${3171.8293*unit_factor}" />
     <xacro:property name="iyy_5" value="${3171.8293*unit_factor}" />
     <xacro:property name="iyy_6" value="${1711.0225*unit_factor}" />
-    <xacro:property name="izz_1" value="${38856.370*unit_factor}" />
-    <xacro:property name="izz_2" value="${1231270.0*unit_factor}" />
-    <xacro:property name="izz_3" value="${135525.91*unit_factor}" />
+    <xacro:property name="izz_1" value="${14241.226*unit_factor}" />
+    <xacro:property name="izz_2" value="${252296.10*unit_factor}" />
+    <xacro:property name="izz_3" value="${36908.834*unit_factor}" />
     <xacro:property name="izz_4" value="${3478.9518*unit_factor}" />
     <xacro:property name="izz_5" value="${3478.9518*unit_factor}" />
@@ -68,11 +68,11 @@
     <visual>
       <geometry>
-        <mesh filename="package://tm_description/meshes/tm12s/visual/tm12s-tbb_a.${format}" />
-      </geometry>
-      <material name="${color}" />
-    </visual>
-    <collision>
-      <geometry>
-        <mesh filename="package://tm_description/meshes/tm12s/collision/tm12s-tbb_a_c.stl" />
+        <mesh filename="package://tm_description/meshes/tm7s/visual/tm7s-base.${format}" />
+      </geometry>
+      <material name="${color}" />
+    </visual>
+    <collision>
+      <geometry>
+        <mesh filename="package://tm_description/meshes/tm7s/collision/tm7s-base_c.stl" />
       </geometry>
     </collision>
@@ -85,5 +85,5 @@
     <parent link="${prefix}link_0" />
     <child link="${prefix}link_1" />
-    <origin rpy="0.000000 -0.000000 0.000000" xyz="0.000000 0.000000 0.165200" />
+    <origin rpy="0.000000 -0.000000 0.000000" xyz="0.000000 0.000000 0.148400" />
     <axis xyz="0 0 1" />
 <!--limit-->
@@ -97,11 +97,11 @@
     <visual>
       <geometry>
-        <mesh filename="package://tm_description/meshes/tm12s/visual/tm12s-j1-a.${format}" />
-      </geometry>
-      <material name="${color}" />
-    </visual>
-    <collision>
-      <geometry>
-        <mesh filename="package://tm_description/meshes/tm12s/collision/tm12s-j1-a_c.stl" />
+        <mesh filename="package://tm_description/meshes/tm7s/visual/tm7s-j1.${format}" />
+      </geometry>
+      <material name="${color}" />
+    </visual>
+    <collision>
+      <geometry>
+        <mesh filename="package://tm_description/meshes/tm7s/collision/tm7s-j1_c.stl" />
       </geometry>
     </collision>
@@ -127,11 +127,11 @@
     <visual>
       <geometry>
-        <mesh filename="package://tm_description/meshes/tm12s/visual/tm12s-a1.${format}" />
-      </geometry>
-      <material name="${color}" />
-    </visual>
-    <collision>
-      <geometry>
-        <mesh filename="package://tm_description/meshes/tm12s/collision/tm12s-a1_c.stl" />
+        <mesh filename="package://tm_description/meshes/tm7s/visual/tm7s-a1.${format}" />
+      </geometry>
+      <material name="${color}" />
+    </visual>
+    <collision>
+      <geometry>
+        <mesh filename="package://tm_description/meshes/tm7s/collision/tm7s-a1_c.stl" />
       </geometry>
     </collision>
@@ -145,5 +145,5 @@
     <parent link="${prefix}link_2" />
     <child link="${prefix}link_3" />
-    <origin rpy="0.000000 -0.000000 0.000000" xyz="0.636100 0.000000 0.000000" />
+    <origin rpy="0.000000 -0.000000 0.000000" xyz="0.329000 0.000000 0.000000" />
     <axis xyz="0 0 1" />
 <!--limit-->
@@ -157,11 +157,11 @@
     <visual>
       <geometry>
-        <mesh filename="package://tm_description/meshes/tm12s/visual/tm12s-a2.${format}" />
-      </geometry>
-      <material name="${color}" />
-    </visual>
-    <collision>
-      <geometry>
-        <mesh filename="package://tm_description/meshes/tm12s/collision/tm12s-a2_c.stl" />
+        <mesh filename="package://tm_description/meshes/tm7s/visual/tm7s-a2.${format}" />
+      </geometry>
+      <material name="${color}" />
+    </visual>
+    <collision>
+      <geometry>
+        <mesh filename="package://tm_description/meshes/tm7s/collision/tm7s-a2_c.stl" />
       </geometry>
     </collision>
@@ -175,5 +175,5 @@
     <parent link="${prefix}link_3" />
     <child link="${prefix}link_4" />
-    <origin rpy="0.000000 -0.000000 1.570796" xyz="0.532400 0.000000 -0.181800" />
+    <origin rpy="0.000000 -0.000000 1.570796" xyz="0.298000 0.000000 -0.147800" />
     <axis xyz="0 0 1" />
 <!--limit-->
@@ -187,11 +187,11 @@
     <visual>
       <geometry>
-        <mesh filename="package://tm_description/meshes/tm12s/visual/tm12s-j5.${format}" />
-      </geometry>
-      <material name="${color}" />
-    </visual>
-    <collision>
-      <geometry>
-        <mesh filename="package://tm_description/meshes/tm12s/collision/tm12s-j5_c.stl" />
+        <mesh filename="package://tm_description/meshes/tm7s/visual/tm7s-j5.${format}" />
+      </geometry>
+      <material name="${color}" />
+    </visual>
+    <collision>
+      <geometry>
+        <mesh filename="package://tm_description/meshes/tm7s/collision/tm7s-j5_c.stl" />
       </geometry>
     </collision>
@@ -217,11 +217,11 @@
     <visual>
       <geometry>
-        <mesh filename="package://tm_description/meshes/tm12s/visual/tm12s-j6.${format}" />
-      </geometry>
-      <material name="${color}" />
-    </visual>
-    <collision>
-      <geometry>
-        <mesh filename="package://tm_description/meshes/tm12s/collision/tm12s-j6_c.stl" />
+        <mesh filename="package://tm_description/meshes/tm7s/visual/tm7s-j6.${format}" />
+      </geometry>
+      <material name="${color}" />
+    </visual>
+    <collision>
+      <geometry>
+        <mesh filename="package://tm_description/meshes/tm7s/collision/tm7s-j6_c.stl" />
       </geometry>
     </collision>
@@ -247,11 +247,11 @@
     <visual>
       <geometry>
-        <mesh filename="package://tm_description/meshes/tm12s/visual/tm12s-io.${format}" />
-      </geometry>
-      <material name="${color}" />
-    </visual>
-    <collision>
-      <geometry>
-        <mesh filename="package://tm_description/meshes/tm12s/collision/tm12s-io_c.stl" />
+        <mesh filename="package://tm_description/meshes/tm7s/visual/tm7s-io.${format}" />
+      </geometry>
+      <material name="${color}" />
+    </visual>
+    <collision>
+      <geometry>
+        <mesh filename="package://tm_description/meshes/tm7s/collision/tm7s-io_c.stl" />
       </geometry>
     </collision>
