Commit message: 1.0.8 Add the TM30S mesh files, Xacro simulation models and update relative joint_velocity_limit values.

File: tm_description/xacro/macro.tm14s-nominal.urdf.xacro (robot description, xacro)
@@ -9,10 +9,10 @@
     wrist_2_joint_lower_limit:=${radians(-360)}    wrist_2_joint_upper_limit:=${radians(360)}
     wrist_3_joint_lower_limit:=${radians(-360)}    wrist_3_joint_upper_limit:=${radians(360)}
-    shoulder_1_joint_velocity_limit:=${radians(160)}
-    shoulder_2_joint_velocity_limit:=${radians(160)}
-    elbow_joint_velocity_limit:=${radians(240)}
-    wrist_1_joint_velocity_limit:=${radians(260)}
-    wrist_2_joint_velocity_limit:=${radians(260)}
-    wrist_3_joint_velocity_limit:=${radians(520)}
+    shoulder_1_joint_velocity_limit:=${radians(130)}
+    shoulder_2_joint_velocity_limit:=${radians(130)}
+    elbow_joint_velocity_limit:=${radians(210)}
+    wrist_1_joint_velocity_limit:=${radians(225)}
+    wrist_2_joint_velocity_limit:=${radians(225)}
+    wrist_3_joint_velocity_limit:=${radians(450)}
     shoulder_1_joint_effort_limit:=${350}
     shoulder_2_joint_effort_limit:=${350}

File: tm_description/xacro/macro.tm25s-nominal.urdf.xacro (robot description, xacro)
@@ -9,10 +9,10 @@
     wrist_2_joint_lower_limit:=${radians(-360)}    wrist_2_joint_upper_limit:=${radians(360)}
     wrist_3_joint_lower_limit:=${radians(-360)}    wrist_3_joint_upper_limit:=${radians(360)}
-    shoulder_1_joint_velocity_limit:=${radians(150)}
-    shoulder_2_joint_velocity_limit:=${radians(150)}
-    elbow_joint_velocity_limit:=${radians(160)}
-    wrist_1_joint_velocity_limit:=${radians(225)}
-    wrist_2_joint_velocity_limit:=${radians(240)}
-    wrist_3_joint_velocity_limit:=${radians(255)}
+    shoulder_1_joint_velocity_limit:=${radians(100)}
+    shoulder_2_joint_velocity_limit:=${radians(100)}
+    elbow_joint_velocity_limit:=${radians(130)}
+    wrist_1_joint_velocity_limit:=${radians(195)}
+    wrist_2_joint_velocity_limit:=${radians(210)}
+    wrist_3_joint_velocity_limit:=${radians(225)}
     shoulder_1_joint_effort_limit:=${750}
     shoulder_2_joint_effort_limit:=${750}

File: tm_description/xacro/macro.tm30s-nominal.urdf.xacro (robot description, xacro)
@@ -2,22 +2,22 @@
 <robot xmlns:xacro="http://www.ros.org/wiki/xacro">
   <xacro:include filename="$(find tm_description)/xacro/macro.inertial.xacro" />
-  <xacro:macro name="tm12s" params="ns prefix color:=none format:=obj
+  <xacro:macro name="tm30s" params="ns prefix color:=none format:=obj
     shoulder_1_joint_lower_limit:=${radians(-360)}    shoulder_1_joint_upper_limit:=${radians(360)}
     shoulder_2_joint_lower_limit:=${radians(-360)}    shoulder_2_joint_upper_limit:=${radians(360)}
-    elbow_joint_lower_limit:=${radians(-162)}    elbow_joint_upper_limit:=${radians(162)}
+    elbow_joint_lower_limit:=${radians(-170)}    elbow_joint_upper_limit:=${radians(170)}
     wrist_1_joint_lower_limit:=${radians(-360)}    wrist_1_joint_upper_limit:=${radians(360)}
     wrist_2_joint_lower_limit:=${radians(-360)}    wrist_2_joint_upper_limit:=${radians(360)}
     wrist_3_joint_lower_limit:=${radians(-360)}    wrist_3_joint_upper_limit:=${radians(360)}
-    shoulder_1_joint_velocity_limit:=${radians(130)}
-    shoulder_2_joint_velocity_limit:=${radians(130)}
-    elbow_joint_velocity_limit:=${radians(210)}
-    wrist_1_joint_velocity_limit:=${radians(225)}
-    wrist_2_joint_velocity_limit:=${radians(225)}
-    wrist_3_joint_velocity_limit:=${radians(450)}
-    shoulder_1_joint_effort_limit:=${350}
-    shoulder_2_joint_effort_limit:=${350}
-    elbow_joint_effort_limit:=${170}
-    wrist_1_joint_effort_limit:=${45}
-    wrist_2_joint_effort_limit:=${45}
+    shoulder_1_joint_velocity_limit:=${radians(100)}
+    shoulder_2_joint_velocity_limit:=${radians(100)}
+    elbow_joint_velocity_limit:=${radians(130)}
+    wrist_1_joint_velocity_limit:=${radians(195)}
+    wrist_2_joint_velocity_limit:=${radians(210)}
+    wrist_3_joint_velocity_limit:=${radians(225)}
+    shoulder_1_joint_effort_limit:=${750}
+    shoulder_2_joint_effort_limit:=${750}
+    elbow_joint_effort_limit:=${350}
+    wrist_1_joint_effort_limit:=${350}
+    wrist_2_joint_effort_limit:=${170}
     wrist_3_joint_effort_limit:=${45}
     safety_limits:=false safety_pos_margin:=0.15
@@ -39,28 +39,28 @@
     <!-- Inertia parameters -->
     <xacro:property name="mass_0" value="1.0" />
-    <xacro:property name="mass_1" value="8.200" />
-    <xacro:property name="mass_2" value="15.017" />
-    <xacro:property name="mass_3" value="3.329" />
-    <xacro:property name="mass_4" value="1.770" />
-    <xacro:property name="mass_5" value="1.880" />
+    <xacro:property name="mass_1" value="22.667" />
+    <xacro:property name="mass_2" value="36.204" />
+    <xacro:property name="mass_3" value="8.028" />
+    <xacro:property name="mass_4" value="6.975" />
+    <xacro:property name="mass_5" value="2.353" />
     <xacro:property name="mass_6" value="0.720" />
     <xacro:property name="unit_factor" value="0.000001"/>
-    <xacro:property name="ixx_1" value="${25963.078*unit_factor}" />
-    <xacro:property name="ixx_2" value="${56178.979*unit_factor}" />
-    <xacro:property name="ixx_3" value="${4694.5431*unit_factor}" />
-    <xacro:property name="ixx_4" value="${2046.0318*unit_factor}" />
-    <xacro:property name="ixx_5" value="${2046.0318*unit_factor}" />
+    <xacro:property name="ixx_1" value="${138058.33*unit_factor}" />
+    <xacro:property name="ixx_2" value="${279146.89*unit_factor}" />
+    <xacro:property name="ixx_3" value="${25838.443*unit_factor}" />
+    <xacro:property name="ixx_4" value="${22651.250*unit_factor}" />
+    <xacro:property name="ixx_5" value="${4938.0363*unit_factor}" />
     <xacro:property name="ixx_6" value="${703.44734*unit_factor}" />
-    <xacro:property name="iyy_1" value="${37671.229*unit_factor}" />
-    <xacro:property name="iyy_2" value="${1212610.4*unit_factor}" />
-    <xacro:property name="iyy_3" value="${134098.54*unit_factor}" />
-    <xacro:property name="iyy_4" value="${3171.8293*unit_factor}" />
-    <xacro:property name="iyy_5" value="${3171.8293*unit_factor}" />
+    <xacro:property name="iyy_1" value="${215387.34*unit_factor}" />
+    <xacro:property name="iyy_2" value="${5261249.9*unit_factor}" />
+    <xacro:property name="iyy_3" value="${36861.092*unit_factor}" />
+    <xacro:property name="iyy_4" value="${266609.58*unit_factor}" />
+    <xacro:property name="iyy_5" value="${5689.9898*unit_factor}" />
     <xacro:property name="iyy_6" value="${1711.0225*unit_factor}" />
-    <xacro:property name="izz_1" value="${38856.370*unit_factor}" />
-    <xacro:property name="izz_2" value="${1231270.0*unit_factor}" />
-    <xacro:property name="izz_3" value="${135525.91*unit_factor}" />
-    <xacro:property name="izz_4" value="${3478.9518*unit_factor}" />
-    <xacro:property name="izz_5" value="${3478.9518*unit_factor}" />
+    <xacro:property name="izz_1" value="${226340.06*unit_factor}" />
+    <xacro:property name="izz_2" value="${5362053.4*unit_factor}" />
+    <xacro:property name="izz_3" value="${38299.020*unit_factor}" />
+    <xacro:property name="izz_4" value="${272336.50*unit_factor}" />
+    <xacro:property name="izz_5" value="${7195.1432*unit_factor}" />
     <xacro:property name="izz_6" value="${1854.4783*unit_factor}" />
 <!--LinkDescription-->
@@ -68,11 +68,11 @@
     <visual>
       <geometry>
-        <mesh filename="package://tm_description/meshes/tm12s/visual/tm12s-tbb_a.${format}" />
-      </geometry>
-      <material name="${color}" />
-    </visual>
-    <collision>
-      <geometry>
-        <mesh filename="package://tm_description/meshes/tm12s/collision/tm12s-tbb_a_c.stl" />
+        <mesh filename="package://tm_description/meshes/tm25s/visual/tm25s-base.${format}" />
+      </geometry>
+      <material name="${color}" />
+    </visual>
+    <collision>
+      <geometry>
+        <mesh filename="package://tm_description/meshes/tm25s/collision/tm25s-base_c.stl" />
       </geometry>
     </collision>
@@ -85,5 +85,5 @@
     <parent link="${prefix}link_0" />
     <child link="${prefix}link_1" />
-    <origin rpy="0.000000 -0.000000 0.000000" xyz="0.000000 0.000000 0.165200" />
+    <origin rpy="0.000000 0.000000 0.000000" xyz="0.000000 0.000000 0.235000" />
     <axis xyz="0 0 1" />
 <!--limit-->
@@ -97,11 +97,11 @@
     <visual>
       <geometry>
-        <mesh filename="package://tm_description/meshes/tm12s/visual/tm12s-j1-a.${format}" />
-      </geometry>
-      <material name="${color}" />
-    </visual>
-    <collision>
-      <geometry>
-        <mesh filename="package://tm_description/meshes/tm12s/collision/tm12s-j1-a_c.stl" />
+        <mesh filename="package://tm_description/meshes/tm25s/visual/tm25s-j1.${format}" />
+      </geometry>
+      <material name="${color}" />
+    </visual>
+    <collision>
+      <geometry>
+        <mesh filename="package://tm_description/meshes/tm25s/collision/tm25s-j1_c.stl" />
       </geometry>
     </collision>
@@ -127,11 +127,11 @@
     <visual>
       <geometry>
-        <mesh filename="package://tm_description/meshes/tm12s/visual/tm12s-a1.${format}" />
-      </geometry>
-      <material name="${color}" />
-    </visual>
-    <collision>
-      <geometry>
-        <mesh filename="package://tm_description/meshes/tm12s/collision/tm12s-a1_c.stl" />
+        <mesh filename="package://tm_description/meshes/tm30s/visual/tm30s-arm1.${format}" />
+      </geometry>
+      <material name="${color}" />
+    </visual>
+    <collision>
+      <geometry>
+        <mesh filename="package://tm_description/meshes/tm30s/collision/tm30s-arm1_c.stl" />
       </geometry>
     </collision>
@@ -145,5 +145,5 @@
     <parent link="${prefix}link_2" />
     <child link="${prefix}link_3" />
-    <origin rpy="0.000000 -0.000000 0.000000" xyz="0.636100 0.000000 0.000000" />
+    <origin rpy="0.000000 0.000000 1.570796" xyz="0.890000 0.000000 -0.070000" />
     <axis xyz="0 0 1" />
 <!--limit-->
@@ -157,11 +157,11 @@
     <visual>
       <geometry>
-        <mesh filename="package://tm_description/meshes/tm12s/visual/tm12s-a2.${format}" />
-      </geometry>
-      <material name="${color}" />
-    </visual>
-    <collision>
-      <geometry>
-        <mesh filename="package://tm_description/meshes/tm12s/collision/tm12s-a2_c.stl" />
+        <mesh filename="package://tm_description/meshes/tm25s/visual/tm25s-j4.${format}" />
+      </geometry>
+      <material name="${color}" />
+    </visual>
+    <collision>
+      <geometry>
+        <mesh filename="package://tm_description/meshes/tm25s/collision/tm25s-j4_c.stl" />
       </geometry>
     </collision>
@@ -175,5 +175,5 @@
     <parent link="${prefix}link_3" />
     <child link="${prefix}link_4" />
-    <origin rpy="0.000000 -0.000000 1.570796" xyz="0.532400 0.000000 -0.181800" />
+    <origin rpy="1.570796 0.000000 0.000000" xyz="0.000000 -0.660000 0.000000" />
     <axis xyz="0 0 1" />
 <!--limit-->
@@ -187,11 +187,11 @@
     <visual>
       <geometry>
-        <mesh filename="package://tm_description/meshes/tm12s/visual/tm12s-j5.${format}" />
-      </geometry>
-      <material name="${color}" />
-    </visual>
-    <collision>
-      <geometry>
-        <mesh filename="package://tm_description/meshes/tm12s/collision/tm12s-j5_c.stl" />
+        <mesh filename="package://tm_description/meshes/tm30s/visual/tm30s-arm2.${format}" />
+      </geometry>
+      <material name="${color}" />
+    </visual>
+    <collision>
+      <geometry>
+        <mesh filename="package://tm_description/meshes/tm30s/collision/tm30s-arm2_c.stl" />
       </geometry>
     </collision>
@@ -205,5 +205,5 @@
     <parent link="${prefix}link_4" />
     <child link="${prefix}link_5" />
-    <origin rpy="1.570796 -0.000000 0.000000" xyz="0.000000 -0.131500 0.000000" />
+    <origin rpy="-1.570796 0.000000 0.000000" xyz="0.000000 0.170200 0.000000" />
     <axis xyz="0 0 1" />
 <!--limit-->
@@ -217,11 +217,11 @@
     <visual>
       <geometry>
-        <mesh filename="package://tm_description/meshes/tm12s/visual/tm12s-j6.${format}" />
-      </geometry>
-      <material name="${color}" />
-    </visual>
-    <collision>
-      <geometry>
-        <mesh filename="package://tm_description/meshes/tm12s/collision/tm12s-j6_c.stl" />
+        <mesh filename="package://tm_description/meshes/tm25s/visual/tm25s-j6.${format}" />
+      </geometry>
+      <material name="${color}" />
+    </visual>
+    <collision>
+      <geometry>
+        <mesh filename="package://tm_description/meshes/tm25s/collision/tm25s-j6_c.stl" />
       </geometry>
     </collision>
@@ -235,5 +235,5 @@
     <parent link="${prefix}link_5" />
     <child link="${prefix}link_6" />
-    <origin rpy="1.570796 -0.000000 0.000000" xyz="0.000000 -0.134950 0.000000" />
+    <origin rpy="1.570796 0.000000 0.000000" xyz="0.000000 -0.152950 0.000000" />
     <axis xyz="0 0 1" />
 <!--limit-->
@@ -247,11 +247,11 @@
     <visual>
       <geometry>
-        <mesh filename="package://tm_description/meshes/tm12s/visual/tm12s-io.${format}" />
-      </geometry>
-      <material name="${color}" />
-    </visual>
-    <collision>
-      <geometry>
-        <mesh filename="package://tm_description/meshes/tm12s/collision/tm12s-io_c.stl" />
+        <mesh filename="package://tm_description/meshes/tm25s/visual/tm25s-io.${format}" />
+      </geometry>
+      <material name="${color}" />
+    </visual>
+    <collision>
+      <geometry>
+        <mesh filename="package://tm_description/meshes/tm25s/collision/tm25s-io_c.stl" />
       </geometry>
     </collision>

File: tm_description/xacro/macro.tm5s-nominal.urdf.xacro (robot description, xacro)
@@ -9,10 +9,10 @@
     wrist_2_joint_lower_limit:=${radians(-360)}    wrist_2_joint_upper_limit:=${radians(360)}
     wrist_3_joint_lower_limit:=${radians(-360)}    wrist_3_joint_upper_limit:=${radians(360)}
-    shoulder_1_joint_velocity_limit:=${radians(240)}
-    shoulder_2_joint_velocity_limit:=${radians(240)}
-    elbow_joint_velocity_limit:=${radians(240)}
-    wrist_1_joint_velocity_limit:=${radians(260)}
-    wrist_2_joint_velocity_limit:=${radians(260)}
-    wrist_3_joint_velocity_limit:=${radians(520)}
+    shoulder_1_joint_velocity_limit:=${radians(210)}
+    shoulder_2_joint_velocity_limit:=${radians(210)}
+    elbow_joint_velocity_limit:=${radians(210)}
+    wrist_1_joint_velocity_limit:=${radians(225)}
+    wrist_2_joint_velocity_limit:=${radians(225)}
+    wrist_3_joint_velocity_limit:=${radians(450)}
     shoulder_1_joint_effort_limit:=${170}
     shoulder_2_joint_effort_limit:=${170}

File: tm_description/xacro/macro.tm7s-nominal.urdf.xacro (robot description, xacro)
@@ -9,10 +9,10 @@
     wrist_2_joint_lower_limit:=${radians(-360)}    wrist_2_joint_upper_limit:=${radians(360)}
     wrist_3_joint_lower_limit:=${radians(-360)}    wrist_3_joint_upper_limit:=${radians(360)}
-    shoulder_1_joint_velocity_limit:=${radians(240)}
-    shoulder_2_joint_velocity_limit:=${radians(240)}
-    elbow_joint_velocity_limit:=${radians(240)}
-    wrist_1_joint_velocity_limit:=${radians(260)}
-    wrist_2_joint_velocity_limit:=${radians(260)}
-    wrist_3_joint_velocity_limit:=${radians(520)}
+    shoulder_1_joint_velocity_limit:=${radians(210)}
+    shoulder_2_joint_velocity_limit:=${radians(210)}
+    elbow_joint_velocity_limit:=${radians(210)}
+    wrist_1_joint_velocity_limit:=${radians(225)}
+    wrist_2_joint_velocity_limit:=${radians(225)}
+    wrist_3_joint_velocity_limit:=${radians(450)}
     shoulder_1_joint_effort_limit:=${170}
     shoulder_2_joint_effort_limit:=${170}
