Commit message: 1.2.0 Add the tm_moveit package, available for TM5S, TM7S, TM12S, TM14S, TM25S, TM30S, and (without the integrated camera) TM5SX, TM7SX, TM12SX, TM14SX, TM25SX, and TM30SX cobot.

File: tm_description/xacro/macro.materials.xacro (robot description, xacro)
@@ -1,44 +1,44 @@
 <?xml version="1.0"?>
 <robot xmlns:xacro="http://www.ros.org/wiki/xacro">
-	<xacro:macro name="tmr_materials">
-		<material name="none">
-			<color rgba="0.0 0.0 0.0 1.0" />
-		</material>
-		<material name="lightgrey">
-			<color rgba="0.5 0.5 0.5 1.0" />
-		</material>
-		<material name="grey">
-			<color rgba="0.75 0.75 0.75 1.0" />
-		</material>
-		<material name="white">
-			<color rgba="0.95 0.95 0.95 1.0" />
-		</material>
-		<material name="red">
-			<color rgba="0.95 0.0 0.0 1.0" />
-		</material>
-		<material name="orange">
-			<color rgba="1.0 0.5 0.0 1.0" />
-		</material>
-		<material name="yellow">
-			<color rgba="1.0 1.0 0.0 1.0" />
-		</material>
-		<material name="green">
-			<color rgba="0.0 1.0 0.0 1.0" />
-		</material>
-		<material name="blue">
-			<color rgba="0.0 0.0 1.0 1.0" />
-		</material>
-		<material name="indigo">
-			<color rgba="0.3 0.3 0.6 1.0" />
-		</material>
-		<material name="violet">
-			<color rgba="0.6 0.0 1.0 1.0" />
-		</material>
-		<material name="black">
-			<color rgba="0.0 0.0 0.0 1.0" />
-		</material>
-		<material name="darkolive">
-			<color rgba="0.3 0.3 0.25 1.0" />
-		</material>
-	</xacro:macro>
+    <xacro:macro name="tmr_materials">
+        <material name="none">
+            <color rgba="0.0 0.0 0.0 1.0" />
+        </material>
+        <material name="lightgrey">
+            <color rgba="0.5 0.5 0.5 1.0" />
+        </material>
+        <material name="grey">
+            <color rgba="0.75 0.75 0.75 1.0" />
+        </material>
+        <material name="white">
+            <color rgba="0.95 0.95 0.95 1.0" />
+        </material>
+        <material name="red">
+            <color rgba="0.95 0.0 0.0 1.0" />
+        </material>
+        <material name="orange">
+            <color rgba="1.0 0.5 0.0 1.0" />
+        </material>
+        <material name="yellow">
+            <color rgba="1.0 1.0 0.0 1.0" />
+        </material>
+        <material name="green">
+            <color rgba="0.0 1.0 0.0 1.0" />
+        </material>
+        <material name="blue">
+            <color rgba="0.0 0.0 1.0 1.0" />
+        </material>
+        <material name="indigo">
+            <color rgba="0.3 0.3 0.6 1.0" />
+        </material>
+        <material name="violet">
+            <color rgba="0.6 0.0 1.0 1.0" />
+        </material>
+        <material name="black">
+            <color rgba="0.0 0.0 0.0 1.0" />
+        </material>
+        <material name="darkolive">
+            <color rgba="0.3 0.3 0.25 1.0" />
+        </material>
+    </xacro:macro>
 </robot>

File: tm_description/xacro/macro.tm12s-nominal.urdf.xacro (robot description, xacro)
@@ -23,18 +23,18 @@
     safety_limits:=false safety_pos_margin:=0.15
     safety_k_position:=20">
-   <xacro:property name="damping_factor" value="0.000"/>
-   <xacro:property name="d1" value="${damping_factor*0.1}"/>
-   <xacro:property name="d2" value="${damping_factor*0.1}"/>
-   <xacro:property name="d3" value="${damping_factor*0.1}"/>
-   <xacro:property name="d4" value="${damping_factor*0.1}"/>
-   <xacro:property name="d5" value="${damping_factor*0.1}"/>
-   <xacro:property name="d6" value="${damping_factor*0.1}"/>
-   <xacro:property name="friction_factor" value="0.000"/>
-   <xacro:property name="f1" value="${friction_factor*0.1}"/>
-   <xacro:property name="f2" value="${friction_factor*0.1}"/>
-   <xacro:property name="f3" value="${friction_factor*0.1}"/>
-   <xacro:property name="f4" value="${friction_factor*0.1}"/>
-   <xacro:property name="f5" value="${friction_factor*0.1}"/>
-   <xacro:property name="f6" value="${friction_factor*0.1}"/>
+    <xacro:property name="damping_factor" value="0.000"/>
+    <xacro:property name="d1" value="${damping_factor*0.1}"/>
+    <xacro:property name="d2" value="${damping_factor*0.1}"/>
+    <xacro:property name="d3" value="${damping_factor*0.1}"/>
+    <xacro:property name="d4" value="${damping_factor*0.1}"/>
+    <xacro:property name="d5" value="${damping_factor*0.1}"/>
+    <xacro:property name="d6" value="${damping_factor*0.1}"/>
+    <xacro:property name="friction_factor" value="0.000"/>
+    <xacro:property name="f1" value="${friction_factor*0.1}"/>
+    <xacro:property name="f2" value="${friction_factor*0.1}"/>
+    <xacro:property name="f3" value="${friction_factor*0.1}"/>
+    <xacro:property name="f4" value="${friction_factor*0.1}"/>
+    <xacro:property name="f5" value="${friction_factor*0.1}"/>
+    <xacro:property name="f6" value="${friction_factor*0.1}"/>
     <!-- Inertia parameters -->
     <xacro:property name="mass_0" value="1.0" />

File: tm_description/xacro/macro.tm14s-nominal.urdf.xacro (robot description, xacro)
@@ -23,18 +23,18 @@
     safety_limits:=false safety_pos_margin:=0.15
     safety_k_position:=20">
-   <xacro:property name="damping_factor" value="0.000"/>
-   <xacro:property name="d1" value="${damping_factor*0.1}"/>
-   <xacro:property name="d2" value="${damping_factor*0.1}"/>
-   <xacro:property name="d3" value="${damping_factor*0.1}"/>
-   <xacro:property name="d4" value="${damping_factor*0.1}"/>
-   <xacro:property name="d5" value="${damping_factor*0.1}"/>
-   <xacro:property name="d6" value="${damping_factor*0.1}"/>
-   <xacro:property name="friction_factor" value="0.000"/>
-   <xacro:property name="f1" value="${friction_factor*0.1}"/>
-   <xacro:property name="f2" value="${friction_factor*0.1}"/>
-   <xacro:property name="f3" value="${friction_factor*0.1}"/>
-   <xacro:property name="f4" value="${friction_factor*0.1}"/>
-   <xacro:property name="f5" value="${friction_factor*0.1}"/>
-   <xacro:property name="f6" value="${friction_factor*0.1}"/>
+    <xacro:property name="damping_factor" value="0.000"/>
+    <xacro:property name="d1" value="${damping_factor*0.1}"/>
+    <xacro:property name="d2" value="${damping_factor*0.1}"/>
+    <xacro:property name="d3" value="${damping_factor*0.1}"/>
+    <xacro:property name="d4" value="${damping_factor*0.1}"/>
+    <xacro:property name="d5" value="${damping_factor*0.1}"/>
+    <xacro:property name="d6" value="${damping_factor*0.1}"/>
+    <xacro:property name="friction_factor" value="0.000"/>
+    <xacro:property name="f1" value="${friction_factor*0.1}"/>
+    <xacro:property name="f2" value="${friction_factor*0.1}"/>
+    <xacro:property name="f3" value="${friction_factor*0.1}"/>
+    <xacro:property name="f4" value="${friction_factor*0.1}"/>
+    <xacro:property name="f5" value="${friction_factor*0.1}"/>
+    <xacro:property name="f6" value="${friction_factor*0.1}"/>
     <!-- Inertia parameters -->
     <xacro:property name="mass_0" value="1.0" />

File: tm_description/xacro/macro.tm25s-nominal.urdf.xacro (robot description, xacro)
@@ -23,18 +23,18 @@
     safety_limits:=false safety_pos_margin:=0.15
     safety_k_position:=20">
-   <xacro:property name="damping_factor" value="0.000"/>
-   <xacro:property name="d1" value="${damping_factor*0.1}"/>
-   <xacro:property name="d2" value="${damping_factor*0.1}"/>
-   <xacro:property name="d3" value="${damping_factor*0.1}"/>
-   <xacro:property name="d4" value="${damping_factor*0.1}"/>
-   <xacro:property name="d5" value="${damping_factor*0.1}"/>
-   <xacro:property name="d6" value="${damping_factor*0.1}"/>
-   <xacro:property name="friction_factor" value="0.000"/>
-   <xacro:property name="f1" value="${friction_factor*0.1}"/>
-   <xacro:property name="f2" value="${friction_factor*0.1}"/>
-   <xacro:property name="f3" value="${friction_factor*0.1}"/>
-   <xacro:property name="f4" value="${friction_factor*0.1}"/>
-   <xacro:property name="f5" value="${friction_factor*0.1}"/>
-   <xacro:property name="f6" value="${friction_factor*0.1}"/>
+    <xacro:property name="damping_factor" value="0.000"/>
+    <xacro:property name="d1" value="${damping_factor*0.1}"/>
+    <xacro:property name="d2" value="${damping_factor*0.1}"/>
+    <xacro:property name="d3" value="${damping_factor*0.1}"/>
+    <xacro:property name="d4" value="${damping_factor*0.1}"/>
+    <xacro:property name="d5" value="${damping_factor*0.1}"/>
+    <xacro:property name="d6" value="${damping_factor*0.1}"/>
+    <xacro:property name="friction_factor" value="0.000"/>
+    <xacro:property name="f1" value="${friction_factor*0.1}"/>
+    <xacro:property name="f2" value="${friction_factor*0.1}"/>
+    <xacro:property name="f3" value="${friction_factor*0.1}"/>
+    <xacro:property name="f4" value="${friction_factor*0.1}"/>
+    <xacro:property name="f5" value="${friction_factor*0.1}"/>
+    <xacro:property name="f6" value="${friction_factor*0.1}"/>
     <!-- Inertia parameters -->
     <xacro:property name="mass_0" value="1.0" />

File: tm_description/xacro/macro.tm30s-nominal.urdf.xacro (robot description, xacro)
@@ -23,18 +23,18 @@
     safety_limits:=false safety_pos_margin:=0.15
     safety_k_position:=20">
-   <xacro:property name="damping_factor" value="0.000"/>
-   <xacro:property name="d1" value="${damping_factor*0.1}"/>
-   <xacro:property name="d2" value="${damping_factor*0.1}"/>
-   <xacro:property name="d3" value="${damping_factor*0.1}"/>
-   <xacro:property name="d4" value="${damping_factor*0.1}"/>
-   <xacro:property name="d5" value="${damping_factor*0.1}"/>
-   <xacro:property name="d6" value="${damping_factor*0.1}"/>
-   <xacro:property name="friction_factor" value="0.000"/>
-   <xacro:property name="f1" value="${friction_factor*0.1}"/>
-   <xacro:property name="f2" value="${friction_factor*0.1}"/>
-   <xacro:property name="f3" value="${friction_factor*0.1}"/>
-   <xacro:property name="f4" value="${friction_factor*0.1}"/>
-   <xacro:property name="f5" value="${friction_factor*0.1}"/>
-   <xacro:property name="f6" value="${friction_factor*0.1}"/>
+    <xacro:property name="damping_factor" value="0.000"/>
+    <xacro:property name="d1" value="${damping_factor*0.1}"/>
+    <xacro:property name="d2" value="${damping_factor*0.1}"/>
+    <xacro:property name="d3" value="${damping_factor*0.1}"/>
+    <xacro:property name="d4" value="${damping_factor*0.1}"/>
+    <xacro:property name="d5" value="${damping_factor*0.1}"/>
+    <xacro:property name="d6" value="${damping_factor*0.1}"/>
+    <xacro:property name="friction_factor" value="0.000"/>
+    <xacro:property name="f1" value="${friction_factor*0.1}"/>
+    <xacro:property name="f2" value="${friction_factor*0.1}"/>
+    <xacro:property name="f3" value="${friction_factor*0.1}"/>
+    <xacro:property name="f4" value="${friction_factor*0.1}"/>
+    <xacro:property name="f5" value="${friction_factor*0.1}"/>
+    <xacro:property name="f6" value="${friction_factor*0.1}"/>
     <!-- Inertia parameters -->
     <xacro:property name="mass_0" value="1.0" />

File: tm_description/xacro/macro.tm5s-nominal.urdf.xacro (robot description, xacro)
@@ -23,18 +23,18 @@
     safety_limits:=false safety_pos_margin:=0.15
     safety_k_position:=20">
-   <xacro:property name="damping_factor" value="0.000"/>
-   <xacro:property name="d1" value="${damping_factor*0.1}"/>
-   <xacro:property name="d2" value="${damping_factor*0.1}"/>
-   <xacro:property name="d3" value="${damping_factor*0.1}"/>
-   <xacro:property name="d4" value="${damping_factor*0.1}"/>
-   <xacro:property name="d5" value="${damping_factor*0.1}"/>
-   <xacro:property name="d6" value="${damping_factor*0.1}"/>
-   <xacro:property name="friction_factor" value="0.000"/>
-   <xacro:property name="f1" value="${friction_factor*0.1}"/>
-   <xacro:property name="f2" value="${friction_factor*0.1}"/>
-   <xacro:property name="f3" value="${friction_factor*0.1}"/>
-   <xacro:property name="f4" value="${friction_factor*0.1}"/>
-   <xacro:property name="f5" value="${friction_factor*0.1}"/>
-   <xacro:property name="f6" value="${friction_factor*0.1}"/>
+    <xacro:property name="damping_factor" value="0.000"/>
+    <xacro:property name="d1" value="${damping_factor*0.1}"/>
+    <xacro:property name="d2" value="${damping_factor*0.1}"/>
+    <xacro:property name="d3" value="${damping_factor*0.1}"/>
+    <xacro:property name="d4" value="${damping_factor*0.1}"/>
+    <xacro:property name="d5" value="${damping_factor*0.1}"/>
+    <xacro:property name="d6" value="${damping_factor*0.1}"/>
+    <xacro:property name="friction_factor" value="0.000"/>
+    <xacro:property name="f1" value="${friction_factor*0.1}"/>
+    <xacro:property name="f2" value="${friction_factor*0.1}"/>
+    <xacro:property name="f3" value="${friction_factor*0.1}"/>
+    <xacro:property name="f4" value="${friction_factor*0.1}"/>
+    <xacro:property name="f5" value="${friction_factor*0.1}"/>
+    <xacro:property name="f6" value="${friction_factor*0.1}"/>
     <!-- Inertia parameters -->
     <xacro:property name="mass_0" value="1.0" />

File: tm_description/xacro/macro.tm7s-nominal.urdf.xacro (robot description, xacro)
@@ -23,18 +23,18 @@
     safety_limits:=false safety_pos_margin:=0.15
     safety_k_position:=20">
-   <xacro:property name="damping_factor" value="0.000"/>
-   <xacro:property name="d1" value="${damping_factor*0.1}"/>
-   <xacro:property name="d2" value="${damping_factor*0.1}"/>
-   <xacro:property name="d3" value="${damping_factor*0.1}"/>
-   <xacro:property name="d4" value="${damping_factor*0.1}"/>
-   <xacro:property name="d5" value="${damping_factor*0.1}"/>
-   <xacro:property name="d6" value="${damping_factor*0.1}"/>
-   <xacro:property name="friction_factor" value="0.000"/>
-   <xacro:property name="f1" value="${friction_factor*0.1}"/>
-   <xacro:property name="f2" value="${friction_factor*0.1}"/>
-   <xacro:property name="f3" value="${friction_factor*0.1}"/>
-   <xacro:property name="f4" value="${friction_factor*0.1}"/>
-   <xacro:property name="f5" value="${friction_factor*0.1}"/>
-   <xacro:property name="f6" value="${friction_factor*0.1}"/>
+    <xacro:property name="damping_factor" value="0.000"/>
+    <xacro:property name="d1" value="${damping_factor*0.1}"/>
+    <xacro:property name="d2" value="${damping_factor*0.1}"/>
+    <xacro:property name="d3" value="${damping_factor*0.1}"/>
+    <xacro:property name="d4" value="${damping_factor*0.1}"/>
+    <xacro:property name="d5" value="${damping_factor*0.1}"/>
+    <xacro:property name="d6" value="${damping_factor*0.1}"/>
+    <xacro:property name="friction_factor" value="0.000"/>
+    <xacro:property name="f1" value="${friction_factor*0.1}"/>
+    <xacro:property name="f2" value="${friction_factor*0.1}"/>
+    <xacro:property name="f3" value="${friction_factor*0.1}"/>
+    <xacro:property name="f4" value="${friction_factor*0.1}"/>
+    <xacro:property name="f5" value="${friction_factor*0.1}"/>
+    <xacro:property name="f6" value="${friction_factor*0.1}"/>
     <!-- Inertia parameters -->
     <xacro:property name="mass_0" value="1.0" />
